Commit message: strip down simulation

File: rr_vehicle_description/urdf/augmented_rc_car.urdf.xacro (robot description, xacro)
@@ -40,16 +40,4 @@
   <xacro:property name="chassis_height" value="0.01"/>
   <xacro:property name="chassis_mass" value="4"/>
-  <!-- battery_dist is the distance between the inner edges of the
-       batteries. battery_comp_depth is the battery compartment depth.
-       battery_length is measured along the x axis, battery_width
-       along the y axis, and battery_height along the z axis. -->
-  <xacro:property name="battery_x_offset" value="0.055"/>
-  <xacro:property name="battery_dist" value="0.065"/>
-  <xacro:property name="battery_comp_depth" value="0.02"/>
-  <xacro:property name="battery_comp_angle" value="0.34906585"/>
-  <xacro:property name="battery_length" value="0.16"/>
-  <xacro:property name="battery_width" value="0.047"/>
-  <xacro:property name="battery_height" value="0.024"/>
-  <xacro:property name="battery_mass" value="0.5025"/>
   <!-- hub_dia and tire_dia are the diameters of the hub and tire,
        respectively. hex_hub_depth is the distance that the hex hub is
@@ -59,6 +47,6 @@
   <xacro:property name="hub_dia" value="0.0826"/>
   <xacro:property name="tire_dia" value="0.107"/>
-  <xacro:property name="tire_width" value="0.0889"/>
-  <xacro:property name="hex_hub_depth" value="0.01445"/>
+  <xacro:property name="tire_width" value="0.0381"/>
+  <xacro:property name="hex_hub_depth" value="0.0091"/>
   <xacro:property name="wheel_mass" value="0.29"/>
   <!-- hex_hub_dist is the distance between left and right hex hubs when
@@ -68,5 +56,5 @@
   <xacro:property name="wheelbase" value="0.335"/>
   <xacro:property name="hex_hub_dist" value="0.365"/>
-  <xacro:property name="axle_length" value="0.03"/>
+  <xacro:property name="axle_length" value="0.01"/>
   <xacro:property name="wheel_travel" value="0.084"/>
   <xacro:property name="shock_z_offset" value="0.0655"/>
@@ -98,7 +86,4 @@
   <!-- ctrl_period is gazebo_ros_control's control period. Unit: hertz. -->
   <xacro:property name="ctrl_period" value="0.01"/>
-  <material name="battery_mat">
-    <color rgba="0 0 1 1"/>
-  </material>
   <material name="chassis_mat">
     <color rgba="0.5 0.5 0.5 1"/>
@@ -145,46 +130,4 @@
                     outer_rad * outer_rad) / 2}"/>
     </inertial>
-  </xacro:macro>
-  <!-- Battery -->
-  <xacro:macro name="battery" params="prefix reflect">
-    <joint name="chassis_to_${prefix}_battery" type="fixed">
-      <parent link="chassis"/>
-      <child link="${prefix}_battery_offset"/>
-      <origin xyz="${battery_x_offset - battery_length / 2}
-                   ${reflect * battery_dist / 2}
-                   0"
-              rpy="${reflect * battery_comp_angle} 0 0"/>
-    </joint>
-    <link name="${prefix}_battery_offset">
-      <xacro:null_inertial/>
-    </link>
-    <joint name="offset_to_${prefix}_battery" type="fixed">
-      <parent link="${prefix}_battery_offset"/>
-      <child link="${prefix}_battery"/>
-      <origin xyz="0
-                   ${reflect * battery_width / 2}
-                   ${(battery_height / 2) - battery_comp_depth}"/>
-    </joint>
-    <link name="${prefix}_battery">
-      <visual>
-        <geometry>
-          <box size="${battery_length} ${battery_width} ${battery_height}"/>
-        </geometry>
-        <material name="battery_mat"/>
-      </visual>
-      <collision>
-        <geometry>
-          <box size="${battery_length} ${battery_width} ${battery_height}"/>
-        </geometry>
-      </collision>
-      <xacro:solid_cuboid_inertial
-         width="${battery_length}" depth="${battery_width}"
-         height="${battery_height}" mass="${battery_mass}">
-        <origin/>
-      </xacro:solid_cuboid_inertial>
-    </link>
-    <gazebo reference="${prefix}_battery">
-      <material>Gazebo/Blue</material>
-    </gazebo>
   </xacro:macro>
   <!-- Shock absorber -->
@@ -336,80 +279,4 @@
     <origin xyz="${chassis_length /2 + 0.12} 0.0 0.0" rpy="0.0 0.0 0.0"/>
    </joint>
-  <link name="eye_link">
-	    <visual>
-	        <geometry>
-	            <box size="0.05 0.1 0.03"/>
-	        </geometry>
-	    </visual>
-	    <collision>
-	        <!-- origin is relative -->
-	        <geometry>
-	            <box size="0.05 0.1 0.03"/>
-	        </geometry>
-	    </collision>
-	</link>
-	  <gazebo reference="eye_link">
-    <material>Gazebo/Red</material>
-  </gazebo>
-	<link name="left_eye">
-	    <visual>
-	        <geometry>
-	            <sphere radius="0.01"/>
-	        </geometry>
-	    </visual>
-	</link>
-	<gazebo reference="left_eye">
-    	<material>Gazebo/Green</material>
-  	</gazebo>
-	<link name="right_eye">
-	    <visual>
-	        <geometry>
-	            <sphere radius="0.01"/>
-	        </geometry>
-	    </visual>
-	</link>
-	<gazebo reference="right_eye">
-    	<material>Gazebo/Green</material>
-  	</gazebo>
-   <joint name="left_eye_to_head" type="fixed">
-    <parent link="eye_link"/>
-    <child link="left_eye"/>
-    <origin xyz="0.03 0.03 0.0" rpy="0.0 0.0 0.0"/>
-   </joint>
-   <joint name="right_eye_to_head" type="fixed">
-    <parent link="eye_link"/>
-    <child link="right_eye"/>
-    <origin xyz="0.03 -0.03 0.0" rpy="0.0 0.0 0.0"/>
-   </joint>
-   <joint name="base_link_to_eye" type="fixed">
-    <parent link="base_link"/>
-    <child link="eye_link"/>
-    <origin xyz="${chassis_length /2 + 0.03} 0.0 0.1" rpy="0.0 0.0 0.0"/>
-   </joint>
-    <joint name="imu_joint" type="fixed">
-		<axis xyz="1 0 0"/>
-		<origin xyz="0 0 0.19"/>
-		<parent link="base_link"/>
-		<child link="imu_link"/>
-	</joint>
-	<link name="imu_link">
-	  <inertial>
-	    <mass value="0.001"/>
-	    <origin rpy="0 0 0" xyz="0 0 0"/>
-	    <inertia ixx="0.0001" ixy="0" ixz="0" iyy="0.000001" iyz="0" izz="0.0001"/>
-	  </inertial>
-	  <visual>
-	    <origin rpy="0 0 0" xyz="0 0 0"/>
-	    <geometry>
-	      <box size="0.001 0.001 0.001"/>
-	    </geometry>
-	  </visual>
-	  <collision>
-	    <origin rpy="0 0 0" xyz="0 0 0"/>
-	    <geometry>
-	      <box size=".001 .001 .001"/>
-	    </geometry>
-	  </collision>
-	</link>
   <!-- Chassis -->
   <link name="chassis">
@@ -440,7 +307,4 @@
     <child link="chassis"/>
   </joint>
-  <!-- Batteries -->
-  <xacro:battery prefix="left" reflect="1"/>
-  <xacro:battery prefix="right" reflect="-1"/>
   <!-- Wheels -->
   <xacro:front_wheel lr_prefix="left" fr_prefix="front"
@@ -461,91 +325,3 @@
     </plugin>
   </gazebo>
-  <!-- Camera left eye-->
-  <gazebo reference="left_eye">
-      <sensor type="camera" name="left_camera">
-          <update_rate>30.0</update_rate>
-          <camera name="head">
-              <horizontal_fov>1.3962634</horizontal_fov>
-              <image>
-                  <width>320</width>
-                  <height>240</height>
-                  <format>R8G8B8</format>
-              </image>
-              <clip>
-                  <near>0.02</near>
-                  <far>300</far>
-              </clip>
-              <noise>
-                  <type>gaussian</type>
-                  <!-- Noise is sampled independently per pixel on each frame.
-                        That pixel's noise value is added to each of its color
-                        channels, which at that point lie in the range [0,1]. -->
-                  <mean>0.0</mean>
-                  <stddev>0.007</stddev>
-              </noise>
-          </camera>
-          <plugin name="camera_controller" filename="libgazebo_ros_camera.so">
-              <alwaysOn>true</alwaysOn>
-              <updateRate>0.0</updateRate>
-              <cameraName>sensors/left_camera</cameraName>
-              <imageTopicName>image_raw</imageTopicName>
-              <cameraInfoTopicName>camera_info</cameraInfoTopicName>
-              <frameName>camera_link</frameName>
-              <hackBaseline>0.07</hackBaseline>
-              <distortionK1>0.0</distortionK1>
-              <distortionK2>0.0</distortionK2>
-              <distortionK3>0.0</distortionK3>
-              <distortionT1>0.0</distortionT1>
-              <distortionT2>0.0</distortionT2>
-          </plugin>
-      </sensor>
-  </gazebo>
-  <!-- Camera right eye-->
-  <gazebo reference="right_eye">
-      <sensor type="camera" name="right_camera">
-          <update_rate>30.0</update_rate>
-          <camera name="head">
-              <horizontal_fov>1.3962634</horizontal_fov>
-              <image>
-                  <width>320</width>
-                  <height>240</height>
-                  <format>R8G8B8</format>
-              </image>
-              <clip>
-                  <near>0.02</near>
-                  <far>300</far>
-              </clip>
-              <noise>
-                  <type>gaussian</type>
-                  <mean>0.0</mean>
-                  <stddev>0.007</stddev>
-              </noise>
-          </camera>
-          <plugin name="camera_controller" filename="libgazebo_ros_camera.so">
-              <alwaysOn>true</alwaysOn>
-              <updateRate>0.0</updateRate>
-              <cameraName>sensors/right_camera</cameraName>
-              <imageTopicName>image_raw</imageTopicName>
-              <cameraInfoTopicName>camera_info</cameraInfoTopicName>
-              <frameName>camera_link</frameName>
-              <hackBaseline>0.07</hackBaseline>
-              <distortionK1>0.0</distortionK1>
-              <distortionK2>0.0</distortionK2>
-              <distortionK3>0.0</distortionK3>
-              <distortionT1>0.0</distortionT1>
-              <distortionT2>0.0</distortionT2>
-          </plugin>
-      </sensor>
-  </gazebo>
-<!-- imu sensor-->
-<gazebo>
-  <plugin name="imu_plugin" filename="libgazebo_ros_imu.so">
-      <alwaysOn>true</alwaysOn>
-      <bodyName>imu_link</bodyName>
-      <topicName>imu_data</topicName>
-      <serviceName>imu_service</serviceName>
-      <gaussianNoise>0.0</gaussianNoise>
-      <updateRate>30.0</updateRate>
-  </plugin>
-</gazebo>
 </robot>

Commit message: removed shock absorbers

File: rr_vehicle_description/urdf/augmented_rc_car.urdf.xacro (robot description, xacro)
@@ -29,5 +29,5 @@
 limitations under the License.
 -->
-<robot name="em_3905" xmlns:xacro="http://www.ros.org/wiki/xacro">
+<robot name="" xmlns:xacro="http://www.ros.org/wiki/xacro">
   <!-- Degree-to-radian conversions -->
   <xacro:property name="degrees_45" value="0.785398163"/>
@@ -35,7 +35,6 @@
   <!-- chassis_length is measured along the x axis, chassis_width
        along the y axis, and chassis_height along the z axis. -->
-  <!--xacro:property name="chassis_length" value="0.258"/-->
   <xacro:property name="chassis_length" value="0.445"/>
-  <xacro:property name="chassis_width" value="0.178"/>
+  <xacro:property name="chassis_width" value="0.165"/>
   <xacro:property name="chassis_height" value="0.01"/>
   <xacro:property name="chassis_mass" value="4"/>
@@ -50,19 +49,7 @@
   <xacro:property name="hex_hub_depth" value="0.0091"/>
   <xacro:property name="wheel_mass" value="0.29"/>
-  <!-- hex_hub_dist is the distance between left and right hex hubs when
-       the shock absorbers are fully extended. axle_length is the distance
-       from a U joint to the corresponding hex hub. wheel_travel is the
-       vertical wheel travel. -->
+  <xacro:property name="axle_length" value="0.01"/>
   <xacro:property name="wheelbase" value="0.335"/>
   <xacro:property name="hex_hub_dist" value="0.365"/>
-  <xacro:property name="axle_length" value="0.01"/>
-  <xacro:property name="wheel_travel" value="0.084"/>
-  <xacro:property name="shock_z_offset" value="0.0655"/>
-  <!-- shock_eff_limit is 2 * ((shock_stroke / 2) * shock_spring_constant) N.
-       shock_stroke is 0.028575 meters. shock_spring_constant, an approximation
-       of a Traxxas Ultra Shock shock absorber spring's constant, is
-       437.817 N/m. -->
-  <xacro:property name="shock_eff_limit" value="12.5106"/>
-  <xacro:property name="shock_vel_limit" value="1000"/>
   <!-- The specifications for a Titan(R) 550 motor could not be found, so the
        stall torque of a Mabuchi Motor(R) RS-550VC-7525 motor was used instead.
@@ -131,27 +118,14 @@
     </inertial>
   </xacro:macro>
-  <!-- Shock absorber -->
+  <!-- Shock absorber without any shock absorption -->
   <xacro:macro name="shock"
                params="lr_prefix fr_prefix lr_reflect fr_reflect child">
-    <joint name="${lr_prefix}_${fr_prefix}_shock" type="prismatic">
+    <joint name="${lr_prefix}_${fr_prefix}_shock" type="fixed">
       <parent link="chassis"/>
       <child link="${child}"/>
       <origin xyz="${fr_reflect * wheelbase / 2}
                    ${lr_reflect * ((hex_hub_dist / 2) - axle_length)}
-                   ${(wheel_travel / 2) - shock_z_offset}"/>
-      <axis xyz="0 0 -1"/>
-      <limit lower="${-wheel_travel / 2}" upper="${wheel_travel / 2}"
-             effort="${shock_eff_limit}" velocity="${shock_vel_limit}"/>
+                   0"/>
     </joint>
-    <transmission name="${lr_prefix}_${fr_prefix}_shock_trans">
-      <type>transmission_interface/SimpleTransmission</type>
-      <joint name="${lr_prefix}_${fr_prefix}_shock">
-        <hardwareInterface>hardware_interface/EffortJointInterface</hardwareInterface>
-      </joint>
-      <actuator name="${lr_prefix}_${fr_prefix}_shock_act">
-        <hardwareInterface>EffortJointInterface</hardwareInterface>
-        <mechanicalReduction>1</mechanicalReduction>
-      </actuator>
-    </transmission>
   </xacro:macro>
   <!-- The "wheel" macro defines an axle carrier, axle, and wheel. -->
@@ -259,24 +233,24 @@
   </gazebo>
   <link name="bumper_link">
-	    <visual>
-	        <geometry>
-	            <box size="0.01 0.3 0.01"/>
-	        </geometry>
-	    </visual>
-	    <collision>
-	        <!-- origin is relative -->
-	        <geometry>
-	            <box size="0.01 0.3 0.01"/>
-	        </geometry>
-	    </collision>
-	</link>
-	<gazebo reference="bumper_link">
-    	<material>Gazebo/Black</material>
-  	</gazebo>
-   <joint name="baselink_to_bumper" type="fixed">
+      <visual>
+          <geometry>
+              <box size="0.01 0.3 0.01"/>
+          </geometry>
+      </visual>
+      <collision>
+          <!-- origin is relative -->
+          <geometry>
+              <box size="0.01 0.3 0.01"/>
+          </geometry>
+      </collision>
+  </link>
+  <gazebo reference="bumper_link">
+    <material>Gazebo/Black</material>
+  </gazebo>
+  <joint name="baselink_to_bumper" type="fixed">
     <parent link="base_link"/>
     <child link="bumper_link"/>
     <origin xyz="${chassis_length /2 + 0.12} 0.0 0.0" rpy="0.0 0.0 0.0"/>
-   </joint>
+  </joint>
   <!-- Chassis -->
   <link name="chassis">

Commit message: add the lidar

File: rr_vehicle_description/urdf/augmented_rc_car.urdf.xacro (robot description, xacro)
@@ -1,2 +1,3 @@
+<?xml version="1.0"?>
 <!--@file augmented_rc_car.urdf.xacro
  -  @brief This file defines a model of the University of
@@ -23,7 +24,4 @@
  -  @competition IARRC 2018
 -->
-<!-- augmented_rc_car.urdf.xacro
--->
-<?xml version="1.0"?>
 <robot name="" xmlns:xacro="http://www.ros.org/wiki/xacro">
   <!-- Degree-to-radian conversions -->
@@ -278,4 +276,23 @@
     <child link="chassis"/>
   </joint>
+  <!-- Outer Shell -->
+  <link name="outer_shell">
+    <inertial>
+      <origin xyz="0.0 0.0 0.0" rpy="0.0 0.0 0.0"/>
+      <mass value="0.1"/>
+      <inertia ixx="0.0" ixy="0.0" ixz="0.0" iyy="0.0" iyz="0.0" izz="0.0"/>
+    </inertial>
+    <visual name="outer_shell_stl">
+      <origin xyz="0.0 0.0 0.0" rpy="0.0 0.0 0.0"/>
+      <geometry>
+        <mesh filename="package://rr_vehicle_description/urdf/RR2018.stl" scale="0.02 0.02 0.02"/>
+      </geometry>
+    </visual>
+  </link>
+  <joint name="chassis_to_outer_shell" type="fixed">
+    <parent link="chassis"/>
+    <child link="outer_shell"/>
+    <origin xyz="-0.26 -0.11 0.05" rpy="${degrees_90} 0.0 ${degrees_90}"/>
+  </joint>
   <!-- Wheels -->
   <xacro:front_wheel lr_prefix="left" fr_prefix="front"
@@ -287,12 +304,63 @@
   <xacro:rear_wheel lr_prefix="right" fr_prefix="rear"
                     lr_reflect="-1" fr_reflect="-1"/>
+  <!-- Sensors -->
+  <!-- Lidar -->
+  <link name="hokuyo_link">
+    <collision>
+      <origin xyz="0 0 0" rpy="0 0 0"/>
+      <geometry>
+        <box size="0.1 0.1 0.1"/>
+      </geometry>
+    </collision>
+    <inertial>
+      <mass value="1e-5" />
+      <origin xyz="0 0 0" rpy="0 0 0"/>
+      <inertia ixx="1e-6" ixy="0" ixz="0" iyy="1e-6" iyz="0" izz="1e-6" />
+    </inertial>
+  </link>
+  <joint name="hokuyo_joint" type="fixed">
+    <origin xyz="0.26 0.0 0.03" rpy="0.0 0.0 0.0"/>
+    <parent link="chassis"/>
+    <child link="hokuyo_link"/>
+  </joint>
+  <!-- ULM-30LX Hokuyo Laser Range Finder -->
+  <gazebo reference="hokuyo_link">
+    <sensor type="ray" name="head_hokuyo_sensor">
+      <pose>0 0 0 0 0 0</pose>
+      <visualize>true</visualize>
+      <update_rate>30</update_rate>
+      <ray>
+        <scan>
+          <horizontal>
+            <samples>1080</samples>
+            <resolution>0.25</resolution>
+            <min_angle>-2.356</min_angle>
+            <max_angle>2.356</max_angle>
+          </horizontal>
+        </scan>
+        <range>
+          <min>0.10</min>
+          <max>30.0</max>
+          <resolution>0.01</resolution>
+        </range>
+        <noise>
+          <type>gaussian</type>
+          <!-- Noise parameters based on published spec for Hokuyo laser
+               achieving "+-30mm" accuracy at range < 10m.  A mean of 0.0m and
+               stddev of 0.01m will put 99.7% of samples within 0.03m of the true
+               reading. -->
+          <mean>0.0</mean>
+          <stddev>0.01</stddev>
+        </noise>
+      </ray>
+      <plugin name="gazebo_ros_head_hokuyo_controller" filename="libgazebo_ros_laser.so">
+        <topicName>laserscan</topicName>
+        <frameName>hokuyo_link</frameName>
+        <robotNamespace>/</robotNamespace>
+      </plugin>
+    </sensor>
+  </gazebo>
   <gazebo>
-    <plugin name="gazebo_ros_control" filename="libgazebo_ros_control.so">
-      <!-- As of 10/7/13, setting controlPeriod to a value greater than
-           Gazebo's simulation period prevents the shock absorbers from
-           working.
-      <controlPeriod>${ctrl_period}</controlPeriod>
-      -->
-    </plugin>
+    <plugin name="gazebo_ros_control" filename="libgazebo_ros_control.so"/>
   </gazebo>
 </robot>

Commit message: add front camera

File: rr_vehicle_description/urdf/augmented_rc_car.urdf.xacro (robot description, xacro)
@@ -319,5 +319,5 @@
     </inertial>
   </link>
-  <joint name="hokuyo_joint" type="fixed">
+  <joint name="chassis_to_hokuyo" type="fixed">
     <origin xyz="0.26 0.0 0.03" rpy="0.0 0.0 0.0"/>
     <parent link="chassis"/>
@@ -361,4 +361,76 @@
     </sensor>
   </gazebo>
+  <!-- Camera -->
+  <xacro:macro name="rr_camera"
+               params="name x_offset y_offset z_offset pitch yaw">
+    <link name="${name}_cam_link">
+      <visual>
+        <geometry>
+          <box size="0.05 0.05 0.05"/>
+        </geometry>
+      </visual>
+      <gazebo reference="${name}_cam_link">
+        <material>Gazebo/Black</material>
+      </gazebo>
+      <collision>
+        <origin xyz="0 0 0" rpy="0 0 0"/>
+        <geometry>
+          <box size="0.1 0.1 0.1"/>
+        </geometry>
+      </collision>
+      <inertial>
+        <mass value="1e-5" />
+        <origin xyz="0 0 0" rpy="0 0 0"/>
+        <inertia ixx="1e-6" ixy="0" ixz="0" iyy="1e-6" iyz="0" izz="1e-6" />
+      </inertial>
+    </link>
+    <joint name="chassis_to_${name}_cam" type="fixed">
+      <origin xyz="${x_offset} ${y_offset} ${z_offset}" rpy="0.0 ${pitch} ${yaw}"/>
+      <parent link="chassis"/>
+      <child link="${name}_cam_link"/>
+    </joint>
+    <gazebo reference="${name}_cam_link">
+      <sensor type="camera" name="${name}_cam">
+        <update_rate>30</update_rate>
+        <camera name="${name}_cam">
+          <horizontal_fov>1.3962634</horizontal_fov>
+          <image>
+            <width>320</width>
+            <height>240</height>
+            <format>R8G8B8</format>
+          </image>
+          <clip>
+            <near>0.02</near>
+            <far>300</far>
+          </clip>
+          <noise>
+            <type>gaussian</type>
+            <!-- Noise is sampled independently per pixel on each frame.
+                That pixel's noise value is added to each of its color
+                channels, which at that point lie in the range [0,1]. -->
+            <mean>0.0</mean>
+            <stddev>0.007</stddev>
+          </noise>
+        </camera>
+        <plugin name="${name}_cam_controller" filename="libgazebo_ros_camera.so">
+          <robotNamespace>/rr_vehicle</robotNamespace>
+          <alwaysOn>true</alwaysOn>
+          <updateRate>0.0</updateRate>
+          <cameraName>${name}_cam</cameraName>
+          <imageTopicName>image_raw</imageTopicName>
+          <cameraInfoTopicName>camera_info</cameraInfoTopicName>
+          <frameName>${name}_cam_link</frameName>
+          <hackBaseline>0.07</hackBaseline>
+          <distortionK1>0.0</distortionK1>
+          <distortionK2>0.0</distortionK2>
+          <distortionK3>0.0</distortionK3>
+          <distortionT1>0.0</distortionT1>
+          <distortionT2>0.0</distortionT2>
+        </plugin>
+      </sensor>
+    </gazebo>
+  </xacro:macro>
+  <xacro:rr_camera name="front_facing" x_offset="0.25"
+                y_offset="0.0" z_offset="0.25" pitch="0.0" yaw="0.0"/>
   <gazebo>
     <plugin name="gazebo_ros_control" filename="libgazebo_ros_control.so"/>
